File: DS3231M/DS3231M.sch (KiCad schematic (older format))
At the start: 13 parts, among them J3 Conn_01x08, U1 DS3231MZ

Commit message: Part number added
Parts:
- U1: Part (none) -> C107410
Changed lines of the file:
@@
 F 2 "Package_SO:SOIC-8_3.9x4.9mm_P1.27mm" H 3125 1800 50  0001 C CNN
 F 3 "http://datasheets.maximintegrated.com/en/ds/DS3231M.pdf" H 3125 1700 50  0001 C CNN
+F 4 "C107410" H 3125 2300 50  0001 C CNN "Part"
 	1    3125 2300
 	1    0    0    -1
